File: termometro_digital_fabricio.kicad_sch (KiCad schematic)
At the start: 27 parts, among them SW1 SW_Push, U1 MT3608, U2 L7805, U3 LM35-LP, U4 ICL7107CPL, U5 ICL7660

Commit message: Uploading files
Parts:
- removed U1: MT3608, Package_TO_SOT_SMD:SOT-23-6, symbol Regulator_Switching:MT3608
- added U1: MT3608, Library:MT3608, symbol New_Library:MT3608
- added U7: 18650, Library:18650, symbol New_Library:18650
- C1, C7: footprint (none) -> Capacitor_THT:CP_Radial_D8.0mm_P5.00mm
- C2: footprint (none) -> Capacitor_THT:CP_Radial_D4.0mm_P1.50mm
- U2: footprint (none) -> Package_TO_SOT_THT:TO-220-3_Vertical
- U5: footprint (none) -> Library:SOIC-8
- U6: footprint (none) -> Library:TP4056
Connections:
- net GND: now also U5.4 (CAP-), U1.4 (OUT-); no longer R7.2
- net VEE: now also R7.2
- net at U5.2 (CAP+): now also C8.1
- net at U5.6 (LV): now also C7.2
- net at U5.7 (OSC): now also C7.1
- net at U2.1 (IN): now also U1.3 (OUT+)
- new net: U6.1 (OUT+), U7.1 (IN+)
- new net: U6.2 (OUT-), U7.2 (IN-)
- new net: U1.1 (IN+), U7.3 (OUT+)
- new net: U1.2 (IN-), U7.4 (OUT-)
Other:
- moved on the sheet: C7, R7
