File: termometro_digital_fabricio.kicad_sch (KiCad schematic)
At the start: 30 parts, among them J1 Conn_01x01_Pin, SW1 SW_Push, U1 MT3608, U2 L7805, U3 LM35-LP, U4 ICL7107CPL, U5 ICL7660, U7 18650

Commit message: Uploading files
Parts:
- U7: footprint Library:BatteryHolder_MPD_BH-18650-PC2 -> Package_TO_SOT_SMD:SOT-23-6
Connections:
- net GND: now also R7.2
- net VEE: no longer R7.2
- net at U6.1 (OUT+): now also U1.1 (IN+), U7.1 (OUT+); no longer U7.3 (IN+)
- net at U6.2 (OUT-): now also U1.2 (IN-), U7.2 (OUT-); no longer U7.4 (IN-)
Other:
- moved on the sheet: U6

Commit message: Uploading files
Parts:
- added J2: Conn_01x02, TerminalBlock_Phoenix:TerminalBlock_Phoenix_MKDS-1,5-2-5.08_1x02_P5.08mm_Horizontal, symbol Connector_Generic:Conn_01x02
Connections:
- net at U1.1 (IN+), U6.1 (OUT+), U7.1 (OUT+): now also J2.1 (Pin_1)
- net at U1.2 (IN-), U6.2 (OUT-), U7.2 (OUT-): now also J2.2 (Pin_2)
Changed lines of the file:
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@@
 	)
 	(junction
+		(at 5.08 29.21)
+		(diameter 0)
+		(color 0 0 0 0)
+	)
+	(junction
 		(at 274.32 128.27)
 		(diameter 0)
@@
 	)
 	(junction
+		(at 2.54 30.48)
+		(diameter 0)
+		(color 0 0 0 0)
+	)
+	(junction
 		(at 53.34 27.94)
 		(diameter 0)
@@
 	(wire
 		(pts
+			(xy 2.54 30.48) (xy 2.54 35.56)
+		)
+		(stroke
+			(width 0)
+			(type default)
+		)
+	)
+	(wire
+		(pts
 			(xy 130.81 76.2) (xy 133.35 76.2)
 		)
@@
 	(wire
 		(pts
-			(xy -5.08 30.48) (xy 17.78 30.48)
+			(xy -5.08 30.48) (xy 2.54 30.48)
 		)
 		(stroke
@@
 	(wire
 		(pts
+			(xy 5.08 29.21) (xy 5.08 35.56)
+		)
+		(stroke
+			(width 0)
+			(type default)
+		)
+	)
+	(wire
+		(pts
 			(xy 240.03 71.12) (xy 240.03 85.09)
 		)
@@
 	(wire
 		(pts
+			(xy 2.54 30.48) (xy 17.78 30.48)
+		)
+		(stroke
+			(width 0)
+			(type default)
+		)
+	)
+	(wire
+		(pts
 			(xy 156.21 25.4) (xy 137.16 25.4)
 		)
@@
 					(unit 1)
 				)
+			)
+		)
+	)
+	(symbol
+		(lib_id "Connector_Generic:Conn_01x02")
+		(at 5.08 40.64 270)
+		(unit 1)
+		(exclude_from_sim no)
+		(in_bom yes)
+		(on_board yes)
+		(dnp no)
+		(fields_autoplaced yes)
+		(property "Reference" "J2"
+			(at 7.62 39.3699 90)
+			(effects
+				(font
+					(size 1.27 1.27)
+				)
+				(justify left)
+			)
+		)
+		(property "Value" "Conn_01x02"
+			(at 7.62 41.9099 90)
+			(effects
+				(font
+					(size 1.27 1.27)
+				)
+				(justify left)
+			)
+		)
+		(property "Footprint" "TerminalBlock_Phoenix:TerminalBlock_Phoenix_MKDS-1,5-2-5.08_1x02_P5.08mm_Horizontal"
+			(at 5.08 40.64 0)
+			(effects
+				(font
+					(size 1.27 1.27)
+				)
+				(hide yes)
+			)
+		)
+		(property "Datasheet" "~"
+			(at 5.08 40.64 0)
+			(effects
+				(font
+					(size 1.27 1.27)
+				)
+				(hide yes)
+			)
+		)
+		(property "Description" "Generic connector, single row, 01x02, script generated (kicad-library-utils/schlib/autogen/connector/)"
+			(at 5.08 40.64 0)
+			(effects
+				(font
+					(size 1.27 1.27)
+				)
+				(hide yes)
+			)
+		)
+		(pin "1"
+		)
+		(pin "2"
+		)
+		(instances
+			(project ""
+				(path "/161d34a1-6999-4fe3-942b-be173cb3f8a5"
+					(reference "J2")
+					(unit 1)
+				)
