File: _autosave-termometro_digital_fabricio.kicad_sch (KiCad schematic)
At the start: 30 parts, among them J1 Conn_01x01_Pin, SW1 SW_Push, U1 MT3608, U2 L7805, U3 LM35-LP, U4 ICL7107CPL, U5 ICL7660, U7 18650

Commit message: Uploading files
Parts:
- U3: footprint Package_TO_SOT_THT:TO-92_Inline -> Package_TO_SOT_THT:TO-92_Inline_Wide
- U7: footprint Library:18650 -> Library:BatteryHolder_MPD_BH-18650-PC2
Connections:
- net at U6.1 (OUT+): now also U7.3 (IN+); no longer U7.1 (IN+)
- net at U6.2 (OUT-): now also U7.4 (IN-); no longer U7.2 (IN-)
- net at U1.1 (IN+): now also U7.1 (OUT+); no longer U7.3 (OUT+)
- net at U1.2 (IN-): now also U7.2 (OUT-); no longer U7.4 (OUT-)
