File: termometro_digital_fabricio.kicad_pcb (KiCad board)
At the start: 2 copper layers, 19 parts, among them SW1 SW_Push, U1 MT3608, U3 LM35-LP, U4 ICL7107CPL

Commit message: Uploading files
Parts:
- added C1: C_Polarized, Capacitor_THT:CP_Radial_D8.0mm_P5.00mm, F.Cu at (203.0, 93.0)
- added C2: 1uF, Capacitor_THT:CP_Radial_D4.0mm_P1.50mm, F.Cu at (193.6, 89.0)
- added C7: C_Polarized, Capacitor_THT:CP_Radial_D8.0mm_P5.00mm, F.Cu at (203.0, 83.5)
- added C8: 1nF, Capacitor_THT:C_Disc_D10.5mm_W5.0mm_P5.00mm, F.Cu at (217.1, 105.1)
- added C9: 0.01uF, Capacitor_THT:C_Disc_D10.5mm_W5.0mm_P7.50mm, F.Cu at (215.9, 111.7)
- added U2: L7805, Package_TO_SOT_THT:TO-220-3_Vertical, F.Cu at (141.1, 98.1)
- added U5: ICL7660, Library:SOIC-8, F.Cu at (138.0, 91.9)
- added U6: ~, Library:TP4056, F.Cu at (221.0, 134.0)
- added U7: 18650, Library:18650, F.Cu at (172.0, 134.0)
- R5: value 100k -> 24K
- U1: footprint Package_TO_SOT_SMD:SOT-23-6 -> Library:MT3608
- moved C5 105.3 mm to (225.0, 83.0), turned to 180 degrees
- moved C6 84.9 mm to (224.0, 72.0), turned to 180 degrees
- moved AFF4 84.4 mm to (33.9, 58.6), turned to 90 degrees
- moved C4 79.7 mm to (223.8, 91.0), turned to 180 degrees
- moved C3 79.6 mm to (223.8, 97.5), turned to 180 degrees
- moved R7 69.5 mm to (84.0, 45.6), turned to 90 degrees
- moved R3 63.0 mm to (168.0, 120.2), turned to 90 degrees
- moved AFF3 61.5 mm to (52.1, 58.6), turned to 90 degrees
- moved R4 60.7 mm to (172.8, 120.2), turned to 90 degrees
- moved RV1 60.1 mm to (204.0, 115.5), turned to 180 degrees
- moved R5 59.2 mm to (177.5, 120.2), turned to 90 degrees
- moved R8 59.1 mm to (191.8, 120.2), turned to 90 degrees
- moved R6 58.4 mm to (182.2, 120.2), turned to 90 degrees
- moved AFF2 38.8 mm to (70.2, 58.6), turned to 90 degrees
- moved U4 37.0 mm to (88.7, 69.5), turned to -90 degrees
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Connections:
- R7 pad 2: GND -> Net-(U4-V-)
- U4 pad 26: VEE -> Net-(U4-V-)
Routing:
- net Net-(AFF3-c): track 0.00 -> 158.7 mm
- net Net-(AFF2-g): track 0.00 -> 146.6 mm
- net Net-(AFF2-f): track 0.00 -> 135.2 mm
- net Net-(AFF2-a): track 0.00 -> 120.8 mm
- net VCC: track 0.00 -> 118.4 mm
- net Net-(AFF3-a): track 0.00 -> 115.3 mm
- net Net-(AFF2-b): track 0.00 -> 108.3 mm
- net Net-(AFF3-g): track 0.00 -> 97.3 mm
- net Net-(AFF3-f): track 0.00 -> 95.4 mm
- net Net-(AFF3-e): track 0.00 -> 88.5 mm
- net Net-(AFF1-g): track 0.00 -> 84.2 mm
- net Net-(AFF1-f): track 0.00 -> 72.9 mm
- net Net-(AFF1-a): track 0.00 -> 59.1 mm
- net Net-(AFF1-b): track 0.00 -> 45.7 mm
- net Net-(AFF3-b): track 0.00 -> 44.0 mm, vias 0 -> 2
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Other:
- board outline added: 100 x 100 mm

Commit message: Uploading files
Parts:
- added J1: Conn_01x01_Pin, Connector_PinHeader_1.00mm:PinHeader_1x01_P1.00mm_Vertical, F.Cu at (199.0, 115.0)
- added R1: 10k, Resistor_THT:R_Axial_DIN0309_L9.0mm_D3.2mm_P15.24mm_Horizontal, F.Cu at (161.4, 122.0)
- C1, C7: value C_Polarized -> 10uF; footprint Capacitor_THT:CP_Radial_D8.0mm_P5.00mm -> Capacitor_THT:CP_Radial_D5.0mm_P2.00mm
- RV1: footprint Potentiometer_THT:Potentiometer_ACP_CA9-H5_Horizontal -> Library:TRIM_3296W-1-250
- U3: footprint Package_TO_SOT_THT:TO-92_Inline -> Package_TO_SOT_THT:TO-92_Inline_Wide
- U5: footprint Library:SOIC-8 -> Package_DIP:DIP-8_W7.62mm_LongPads
- U7: footprint Library:18650 -> Library:BatteryHolder_MPD_BH-18650-PC2
- moved AFF4 123.2 mm to (155.9, 75.6)
- moved AFF3 121.2 mm to (172.1, 75.6)
- moved AFF2 119.7 mm to (188.7, 75.6)
- moved R7 119.3 mm to (202.0, 63.0)
- moved AFF1 118.2 mm to (205.4, 75.6)
- moved U4 118.2 mm to (205.7, 86.5)
- moved U3 104.1 mm to (226.0, 123.9), turned to -90 degrees
- moved U2 95.1 mm to (225.8, 141.4), turned to 90 degrees
- moved U5 88.6 mm to (216.5, 133.0), turned to -90 degrees
- moved SW1 79.3 mm to (219.8, 95.8), turned to 0 degrees
- moved U6 79.0 mm to (142.0, 134.0)
- moved U7 70.1 mm to (141.2, 71.0), turned to -90 degrees
- moved C5 58.1 mm to (181.0, 121.0), turned to 0 degrees
- moved C7 56.0 mm to (204.8, 139.4)
- moved C3 53.3 mm to (173.0, 113.8), turned to 90 degrees
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Connections:
- C1 pad 1: Net-(U4-V-) -> VEE
- C7 pad 1: Net-(U5-OSC) -> Net-(U5-CAP+)
- C7 pad 2: Net-(U5-LV) -> Net-(U5-CAP-)
- C8 pad 1: Net-(U5-CAP+) -> Net-(U5-OSC)
- R7 pad 2: Net-(U4-V-) -> VEE
- U4 pad 26: Net-(U4-V-) -> VEE
- U5 pad 4: GND -> Net-(U5-CAP-)
- U5 pad 5: VCC -> VEE
- U5 pad 6: Net-(U5-LV) -> GND
- U5 pad 8: Net-(U4-V-) -> VCC
Routing:
- net VCC: track 118.4 -> 393.9 mm, vias 0 -> 3
- net VEE: track 0.00 -> 275.0 mm
- net GND: track 36.7 -> 253.0 mm, vias 0 -> 2
- net Net-(U4-TEST): track 0.00 -> 48.9 mm
- net Net-(U1-OUT+): track 0.00 -> 47.4 mm
- net Net-(R5-Pad2): track 0.00 -> 42.7 mm
- net Net-(U5-OSC): track 0.00 -> 38.2 mm
- net Net-(C3-Pad1): track 0.00 -> 37.9 mm
- net Net-(U4-BUFF): track 0.00 -> 29.0 mm
- net Net-(U4-IN_HI): track 0.00 -> 28.2 mm
- net Net-(J1-Pin_1): track 0.00 -> 27.7 mm
- net Net-(U4-A-Z): track 0.00 -> 27.4 mm
- net Net-(U1-IN+): track 0.00 -> 26.4 mm
- net Net-(U4-OSC1): track 0.00 -> 23.2 mm
- net Net-(U4-CREF-): track 0.00 -> 23.0 mm
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
Commit message: Uploading files
Parts:
- moved R4 1.58 mm to (154.5, 127.1)
- moved U7 1.28 mm to (142.0, 70.0)
Routing:
- net Net-(C3-Pad1): track 37.9 -> 36.2 mm
- net Net-(U1-IN-): track 17.1 -> 15.9 mm
- net Net-(U1-IN+): track 26.4 -> 25.2 mm
- net Net-(U4-BUFF): track 29.0 -> 27.9 mm
- net Net-(AFF2-f): track 136.3 -> 135.5 mm
- net VEE: track 275.0 -> 274.4 mm

Commit message: Uploading files
Other:
- board text added: "Termômetro Digital Fabricio Rodrigues"
Changed lines of the file:
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@@
 		(layer "Edge.Cuts")
+	)
+	(gr_text "Termômetro Digital\nFabricio Rodrigues"
+		(at 131.5 51 0)
+		(layer "F.SilkS")
+		(effects
+			(font
+				(size 1.5 1.5)
+				(thickness 0.3)
+				(bold yes)
+			)
+			(justify left bottom)
+		)
 	)
 	(segment

Commit message: Uploading files
Parts:
- moved U6 79.0 mm to (143.0, 55.0), turned to 0 degrees
- moved U7 71.0 mm to (142.0, 141.0), turned to 90 degrees
Connections:
- R7 pad 2: VEE -> GND
Routing:
- net GND: track 253.0 -> 466.4 mm
- net VEE: track 274.4 -> 119.3 mm
- net Net-(U1-IN-): track 15.9 -> 129.2 mm
- net Net-(U1-IN+): track 25.2 -> 100.7 mm
- added copper zone on B.Cu, net GND

Commit message: Uploading files
Parts:
- added J2: Conn_01x02, TerminalBlock_Phoenix:TerminalBlock_Phoenix_MKDS-1,5-2-5.08_1x02_P5.08mm_Horizontal, F.Cu at (140.9, 139.0)
Connections:
- U1 pad 1: Net-(U1-IN+) -> Net-(J2-Pin_1)
- U1 pad 2: Net-(U1-IN-) -> Net-(J2-Pin_2)
- U6 pad 1: Net-(U1-IN+) -> Net-(J2-Pin_1)
- U6 pad 2: Net-(U1-IN-) -> Net-(J2-Pin_2)
Routing:
- net Net-(J2-Pin_1): track 0.00 -> 18.8 mm
- net Net-(J2-Pin_2): track 0.00 -> 11.5 mm
